File: pcb/Rev1.sch (EAGLE design)
At the start: 12 parts, among them IC1 74LS595N, IC10 74LS595N, IC11 74LS595N, IC12 74LS595N, IC3 74LS595N, IC4 74LS595N, IC5 74LS595N, IC6 74LS595N, IC7 74LS595N, IC8 74LS595N, IC9 74LS595N

Commit message: <djfhasliughadilfughasdf
Parts:
- added JP10, JP11, JP12, JP2, JP3, JP4, JP5, JP6, JP7, JP8, JP9: (no value), SparkFun-Connectors:M07
Connections:
- new net N$13: IC12.QB, JP2.1
- new net N$14: IC12.QC, JP2.2
- new net N$15: IC12.QD, JP2.3
- new net N$16: IC12.QE, JP2.4
- new net N$17: IC12.QF, JP2.5
- new net N$18: IC12.QG, JP2.6
- new net N$19: IC12.QH, JP2.7
- new net N$20: IC11.QB, JP3.1
- new net N$21: IC11.QC, JP3.2
- new net N$22: IC11.QD, JP3.3
- new net N$23: IC11.QE, JP3.4
- new net N$24: IC11.QF, JP3.5
- new net N$25: IC11.QG, JP3.6
- new net N$26: IC11.QH, JP3.7
- new net N$27: IC10.QB, JP4.1
- new net N$28: IC10.QC, JP4.2
- new net N$29: IC10.QD, JP4.3
- new net N$30: IC10.QE, JP4.4
- new net N$31: IC10.QF, JP4.5
- new net N$32: IC10.QG, JP4.6
- new net N$33: IC10.QH, JP4.7
- new net N$34: IC5.QB, JP5.1
- new net N$35: IC5.QC, JP5.2
- new net N$36: IC5.QD, JP5.3
- new net N$37: IC5.QE, JP5.4
- new net N$38: IC5.QF, JP5.5
- new net N$39: IC5.QG, JP5.6
- new net N$40: IC5.QH, JP5.7
- new net N$41: IC3.QB, JP7.1
- new net N$42: IC3.QC, JP7.2
- new net N$43: IC3.QD, JP7.3
- new net N$44: IC3.QE, JP7.4
- new net N$45: IC3.QF, JP7.5
- new net N$46: IC3.QG, JP7.6
- new net N$47: IC3.QH, JP7.7
- new net N$48: IC4.QB, JP8.1
- new net N$49: IC4.QC, JP8.2
- new net N$50: IC4.QD, JP8.3
- new net N$51: IC4.QE, JP8.4
- new net N$52: IC4.QF, JP8.5
- new net N$53: IC4.QG, JP8.6
- new net N$54: IC4.QH, JP8.7
- new net N$55: IC6.QB, JP9.1
- new net N$56: IC6.QC, JP9.2
- new net N$57: IC6.QD, JP9.3
- new net N$58: IC6.QE, JP9.4
- new net N$59: IC6.QF, JP9.5
- new net N$60: IC6.QG, JP9.6
- new net N$61: IC6.QH, JP9.7
- new net N$62: IC7.QB, JP10.1
- new net N$63: IC7.QC, JP10.2
- new net N$64: IC7.QD, JP10.3
- new net N$65: IC7.QE, JP10.4
- new net N$66: IC7.QF, JP10.5
- new net N$67: IC7.QG, JP10.6
- new net N$68: IC7.QH, JP10.7
- new net N$69: IC8.QB, JP11.1
- new net N$7: IC3.QH*, IC4.SER
- new net N$70: IC8.QC, JP11.2
- new net N$71: IC8.QD, JP11.3
- new net N$72: IC8.QE, JP11.4
- new net N$73: IC8.QF, JP11.5
- new net N$74: IC8.QG, JP11.6
- new net N$75: IC8.QH, JP11.7
- new net N$76: IC9.QB, JP12.1
- new net N$77: IC9.QC, JP12.2
- new net N$78: IC9.QD, JP12.3
- new net N$79: IC9.QE, JP12.4
- new net N$80: IC9.QF, JP12.5
- new net N$81: IC9.QG, JP12.6
- new net N$82: IC9.QH, JP12.7
- new net N$83: IC1.QB, JP6.1
- new net N$84: IC1.QC, JP6.2
- new net N$85: IC1.QD, JP6.3
- new net N$86: IC1.QE, JP6.4
- new net N$87: IC1.QF, JP6.5
- new net N$88: IC1.QG, JP6.6
- new net N$89: IC1.QH, JP6.7
- net GROUND: now also IC1.GND, IC11.GND, IC12.GND, IC3.GND, IC4.GND, IC5.GND, IC8.GND
- net LATCH: now also IC3.RCK, IC5.RCK
- net N$10: now also IC7.QH*
- net N$12: now also IC1.SCK, IC10.SCK, IC12.SCK, IC3.SCK, IC5.SCK, IC6.SCK, IC8.SCK, IC9.SCK
- net N$3: now also IC11.QH*
- net N$6: now also IC1.QH*
- net N$9: now also IC6.QH*
- net VCC: now also IC1.SCL, IC1.VCC, IC10.SCL, IC10.VCC, IC11.VCC, IC12.SCL, IC3.SCL, IC3.VCC, IC4.VCC, IC5.VCC, IC6.SCL, IC6.VCC, IC7.VCC, IC9.SCL
Other:
- moved on the sheet: IC1
